File: project/project.kicad_pcb (KiCad board)
At the start: 2 copper layers, 22 parts, among them U2 NE555P, U4 ROB-14450

Commit message: Add files via upload
Parts:
- moved R5 0.16 mm to (129.0, 46.7)
- renumbered TB1 to NANO, U2 to NE555, U4 to TB6612
Changed lines of the file:
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@@
 		(tags "resistor")
 		(property "Reference" "R1"
-			(at -2.5875 0 360)
+			(at -3.24 0 360)
 			(layer "F.SilkS")
 			(effects
@@
 		(tags "resistor")
 		(property "Reference" "R4"
-			(at -0.5875 1.765 90)
+			(at 0.284477 2.1325 90)
 			(layer "F.SilkS")
-			(hide yes)
 			(effects
 				(font
@@
 		(tags "capacitor")
 		(property "Reference" "C3"
-			(at -0.55 -2 360)
+			(at 0.95 -2.56 360)
 			(layer "F.SilkS")
-			(hide yes)
 			(effects
 				(font
@@
 			(layer "F.Fab")
 		)
-		(fp_text user "${REFERENCE}"
-			(at 0 0 360)
-			(layer "F.Fab")
-			(effects
-				(font
-					(size 0.5 0.5)
-					(thickness 0.08)
-				)
-			)
-		)
 		(pad "1" smd roundrect
 			(at -0.95 0 180)
@@
 	(footprint "Resistor_SMD:R_0805_2012Metric"
 		(layer "F.Cu")
-		(at 129.1325 46.628023 -90)
+		(at 129 46.715523 -90)
 		(descr "Resistor SMD 0805 (2012 Metric), square (rectangular) end terminal, IPC_7351 nominal, (Body size source: IPC-SM-782 page 72, https://www.pcb-3d.com/wordpress/wp-content/uploads/ipc-sm-782a_amendment_1_and_2.pdf), generated with kicad-footprint-generator")
 		(tags "resistor")
 		(property "Reference" "R5"
-			(at 0 2.265 90)
+			(at 2.5875 0 360)
 			(layer "F.SilkS")
-			(hide yes)
 			(effects
 				(font
@@
 		)
 		(property "Value" "R"
-			(at 77.2125 37.0875 360)
+			(at 77.2125 37.0875 0)
 			(layer "F.Fab")
 			(hide yes)
@@
 		(tags "resistor")
 		(property "Reference" "R6"
-			(at 0 1.5 90)
+			(at 2.4675 0 180)
 			(layer "F.SilkS")
-			(hide yes)
 			(effects
 				(font
@@
 		(tags "capacitor")
 		(property "Reference" "C1"
-			(at -2.55 0 180)
+			(at -2.67 -0.5 180)
 			(layer "F.SilkS")
 			(effects
@@
 		(layer "F.Cu")
 		(at 119 90.75)
-		(property "Reference" "U4"
+		(property "Reference" "TB6612"
 			(at -5.5332 -11.6132 360)
 			(layer "F.SilkS")
@@
 			(at -0.9125 2 90)
 			(layer "F.SilkS")
-			(hide yes)
 			(effects
 				(font
@@
 		(descr "Arduino Nano, http://www.mouser.com/pdfdocs/Gravitech_Arduino_Nano3_0.pdf")
 		(tags "Arduino Nano")
-		(property "Reference" "TB1"
+		(property "Reference" "NANO"
 			(at 7.62 -5.08 360)
 			(layer "F.SilkS")
-			(hide yes)
 			(effects
 				(font
@@
 			(at 8.89 19.05 90)
 			(layer "F.Fab")
+			(hide yes)
 			(effects
 				(font
@@
 		(tags "LED diameter 5.0mm 2 pins")
 		(property "Reference" "D4"
-			(at 1.27 4 60)
+			(at 1.605563 4.003599 60)
 			(layer "F.SilkS")
 			(effects
@@
 		(tags "resistor")
 		(property "Reference" "R9"
-			(at 0.0875 1.735 90)
+			(at 1.284477 1.735 90)
 			(layer "F.SilkS")
-			(hide yes)
 			(effects
 				(font
@@
 		(descr "8-lead though-hole mounted DIP package, row spacing 7.62 mm (300 mils)")
 		(tags "THT DIP DIL PDIP 2.54mm 7.62mm 300mil")
-		(property "Reference" "U2"
+		(property "Reference" "NE555"
 			(at 3.81 -2.33 90)
 			(layer "F.SilkS")
-			(hide yes)
 			(effects
 				(font
@@
 			(at 3.81 9.95 90)
 			(layer "F.Fab")
-			(hide yes)
 			(effects
 				(font
@@
 		(tags "resistor")
 		(property "Reference" "R8"
-			(at -0.9125 1.5 90)
+			(at 1.196977 -1.8675 90)
 			(layer "F.SilkS")
-			(hide yes)
 			(effects
 				(font
@@
 	)
 	(segment
-		(start 129.1325 45.715523)
-		(end 129.1325 44.443546)
+		(start 129 44.311046)
+		(end 129 45.803023)
 		(width 1.5)
 		(layer "F.Cu")
@@
 	)
 	(segment
-		(start 129.1325 44.443546)
-		(end 126 41.311046)
+		(start 126 41.311046)
+		(end 129 44.311046)
 		(width 1.5)
 		(layer "F.Cu")

Commit message: Add files via upload
Parts:
- removed D5, D6, D7, D8: LED, LED_THT:LED_D5.0mm
- removed R6, R7, R8, R9: R, Resistor_SMD:R_0805_2012Metric
- added J1: Conn_01x03_Pin, Connector_PinSocket_2.00mm:PinSocket_1x03_P2.00mm_Vertical, F.Cu at (106.5, 59.0)
- added J2: Conn_01x03_Pin, Connector_PinSocket_2.00mm:PinSocket_1x03_P2.00mm_Vertical, F.Cu at (129.5, 39.0)
- added J3: Conn_01x03_Pin, Connector_PinSocket_2.00mm:PinSocket_1x03_P2.00mm_Vertical, F.Cu at (137.0, 42.5)
- added J4: Conn_01x03_Pin, Connector_PinSocket_2.00mm:PinSocket_1x03_P2.00mm_Vertical, F.Cu at (161.5, 59.5)
- added R10: R, Resistor_SMD:R_0805_2012Metric, F.Cu at (131.5, 66.0)
- moved D3 9.87 mm to (140.5, 47.3)
- moved D4 8.97 mm to (123.0, 47.0)
- moved R4 3.72 mm to (136.0, 50.4)
- moved R5 3.43 mm to (128.0, 50.0)
- moved R1 2.26 mm to (137.5, 65.8)
- moved R3 1.50 mm to (112.5, 64.0)
- moved D1 1.00 mm to (114.5, 58.1), turned to 175 degrees
- moved D2 0.64 mm to (149.5, 58.7), turned to 5 degrees
- renumbered NANO to TB1, NE555 to U2, TB6612 to U4
Connections:
- U2 pad 3: Net-(D1-K) -> unconnected-(U2-Q-Pad3)
Routing:
- net GND: track 66.9 -> 187.4 mm
- net Net-(J2-Pin_2): track 123.8 -> 105.7 mm
- net Net-(J3-Pin_2): track 75.1 -> 85.8 mm
- net Net-(D4-A): track 5.73 -> 0.00 mm
- net Net-(D8-A): track 5.16 -> 0.00 mm
- net Net-(D7-A): track 5.02 -> 0.00 mm
- net Net-(D6-A): track 5.01 -> 0.00 mm
- net Net-(D5-A): track 4.69 -> 0.00 mm
- net +5V: track 192.7 -> 196.8 mm
- net Net-(U2-DIS): track 2.81 -> 6.70 mm
- net Net-(U2-THR): track 15.9 -> 19.1 mm
- net Net-(J1-Pin_2): track 148.6 -> 151.5 mm
- net Net-(D1-K): track 70.5 -> 73.0 mm
- net Net-(J4-Pin_2): track 41.8 -> 39.7 mm
- net Net-(D3-A): track 4.75 -> 5.77 mm
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Other:
- board text removed: "${REFERENCE}"
